File: libra-cervisiae-pcb/libra-cervisiae-pcb.sch (KiCad schematic (older format))
At the start: 32 parts, among them CN1 CP2102-BREAKOUT, CN2 TP4056, CN3 HX711_BREAKOUT, J10 Load Cell, J12 Load Cell, J3 Battery, J4 DS18B20, J8 Load Cell, J9 Load Cell, Q1 AO3401, SW1 Reset, SW2 Flash, U1 VREG, U2 ESP-12F

Commit message: Libra Cervisiae logo, relayout
Connections:
- net labels added: E+, E-, S+, S-
- net labels removed: BLK, GRN, RED, WHT
Changed lines of the file:
@@
 encoding utf-8
 Sheet 1 1
-Title "Pendulum PCB"
-Date "2018-06-28"
-Rev "1.0.0-rc.7"
+Title "Libra Cervisiae PCB"
+Date "2018-07-19"
+Rev "1.0.0-rc.1"
 Comp ""
 Comment1 ""
@@
 	1150 4750 1450 4750
 Text Label 8950 5450 0    60   ~ 0
-GRN
+S+
 Text Label 8950 5550 0    60   ~ 0
-WHT
+S-
 Text Label 8950 5650 0    60   ~ 0
-BLK
+E-
 Text Label 8950 5750 0    60   ~ 0
-RED
+E+
 Wire Wire Line
 	3950 5400 3200 5400
@@
 	10100 5750 9950 5750
 Text Label 9950 5450 0    60   ~ 0
-GRN
+S+
 Text Label 9950 5550 0    60   ~ 0
-WHT
+S-
 Text Label 9950 5650 0    60   ~ 0
-BLK
+E-
 Text Label 9950 5750 0    60   ~ 0
-RED
+E+
 Wire Wire Line
 	8950 5450 9150 5450
@@
 	10100 6350 9950 6350
 Text Label 9950 6050 0    60   ~ 0
-GRN
+S+
 Text Label 9350 5450 0    60   ~ 0
-GRN
+S+
 Text Label 9350 6050 0    60   ~ 0
-GRN
+S+
 Text Label 9350 5550 0    60   ~ 0
-WHT
+S-
 Text Label 9350 6150 0    60   ~ 0
-WHT
+S-
 Text Label 9950 6150 0    60   ~ 0
-WHT
+S-
 Text Label 9350 5650 0    60   ~ 0
-BLK
+E-
 Text Label 9350 6250 0    60   ~ 0
-BLK
+E-
 Text Label 9950 6250 0    60   ~ 0
-BLK
+E-
 Text Label 9350 5750 0    60   ~ 0
-RED
+E+
 Text Label 9350 6350 0    60   ~ 0
-RED
+E+
 Text Label 9950 6350 0    60   ~ 0
-RED
+E+
 Wire Wire Line
 	3200 5600 3950 5600

Commit message: Libra Cervisiae: add a temperature sensor to the board
Optional, but recommended: can be used to correct load cell
output for ambient temperature changes.
Parts:
- added J1: Board Temp, Package_TO_SOT_THT:TO-92, symbol conn:Conn_01x03
- J4: value DS18B20 -> Wort Temp
Connections:
- wire segments 142 -> 153
Other:
- note added: "DS18B20s"
- note removed: "DS18B20"
Changed lines of the file:
@@
 Text Label 1950 5900 0    60   ~ 0
 DS+
-Text Label 2100 6100 2    60   ~ 0
+Text Label 1950 6100 0    60   ~ 0
 GND
 $Comp
@@
 P 950 6000
 F 0 "J4" H 950 6200 50  0000 C CNN
-F 1 "DS18B20" H 950 5800 50  0000 C CNN
+F 1 "Wort Temp" H 950 5800 50  0000 C CNN
 F 2 "Connector_Molex:Molex_PicoBlade_53048-0610_1x03_P1.25mm_Horizontal" H 950 6000 50  0001 C CNN
 F 3 "" H 950 6000 50  0001 C CNN
@@
 $EndComp
 Text Notes 1250 5700 0    60   ~ 0
-DS18B20
+DS18B20s
 $Comp
 L hx711_breakout:HX711_BREAKOUT CN3
@@
 L device:C C4
 U 1 1 5B2A9325
-P 1350 6200
-F 0 "C4" V 1400 6050 50  0000 L CNN
-F 1 "1uF" V 1500 6150 50  0000 L CNN
-F 2 "Capacitor_SMD:C_0805_2012Metric" H 1388 6050 50  0001 C CNN
-F 3 "" H 1350 6200 50  0001 C CNN
-	1    1350 6200
+P 1350 6450
+F 0 "C4" V 1400 6300 50  0000 L CNN
+F 1 "1uF" V 1500 6400 50  0000 L CNN
+F 2 "Capacitor_SMD:C_0805_2012Metric" H 1388 6300 50  0001 C CNN
+F 3 "" H 1350 6450 50  0001 C CNN
+	1    1350 6450
 	0    1    1    0
 $EndComp
@@
 L device:R R9
 U 1 1 5B4177F1
-P 1750 6200
-F 0 "R9" V 1830 6200 50  0000 C CNN
-F 1 "10k" V 1750 6200 50  0000 C CNN
-F 2 "Resistor_SMD:R_0805_2012Metric" V 1680 6200 50  0001 C CNN
-F 3 "" H 1750 6200 50  0001 C CNN
-	1    1750 6200
+P 1750 6450
+F 0 "R9" V 1830 6450 50  0000 C CNN
+F 1 "10k" V 1750 6450 50  0000 C CNN
+F 2 "Resistor_SMD:R_0805_2012Metric" V 1680 6450 50  0001 C CNN
+F 3 "" H 1750 6450 50  0001 C CNN
+	1    1750 6450
 	0    1    1    0
 $EndComp
@@
 	1150 5900 1200 5900
 Wire Wire Line
-	1200 5900 1200 6200
-Wire Wire Line
 	1150 6100 1500 6100
 Connection ~ 1200 5900
 Wire Wire Line
 	1200 5900 1600 5900
-Wire Wire Line
-	1500 6200 1500 6100
 Connection ~ 1500 6100
 Wire Wire Line
 	1500 6100 2100 6100
-Wire Wire Line
-	1600 5900 1600 6200
 Connection ~ 1600 5900
 Wire Wire Line
 	1600 5900 2100 5900
-Wire Wire Line
-	1900 6200 1900 6000
 Connection ~ 1900 6000
 Wire Wire Line
@@
 Text Label 3450 2050 1    60   ~ 0
 BAT-
+$Comp
+L conn:Conn_01x03 J1
+U 1 1 5B523E0B
+P 950 6950
+F 0 "J1" H 950 7150 50  0000 C CNN
+F 1 "Board Temp" H 950 6750 50  0000 C CNN
+F 2 "Package_TO_SOT_THT:TO-92" H 950 6950 50  0001 C CNN
+F 3 "" H 950 6950 50  0001 C CNN
+	1    950  6950
+	-1   0    0    1
+$EndComp
+Wire Wire Line
+	1200 5900 1200 6450
+Wire Wire Line
+	1500 6100 1500 6450
+Wire Wire Line
+	1150 6850 1200 6850
+Wire Wire Line
+	1150 7050 1500 7050
+Text Label 1950 6850 0    60   ~ 0
+DS+
+Text Label 1950 6950 0    60   ~ 0
+DSD
+Text Label 1950 7050 0    60   ~ 0
+GND
+Wire Wire Line
+	1200 6450 1200 6850
+Connection ~ 1200 6450
+Connection ~ 1200 6850
+Wire Wire Line
+	1500 6450 1500 7050
+Connection ~ 1500 6450
+Connection ~ 1500 7050
+Wire Wire Line
+	1500 7050 2100 7050
+Wire Wire Line
+	1150 6950 1900 6950
+Wire Wire Line
+	1200 6850 1600 6850
+Wire Wire Line
+	1600 5900 1600 6450
+Wire Wire Line
+	1600 6450 1600 6850
+Connection ~ 1600 6450
+Connection ~ 1600 6850
+Wire Wire Line
+	1600 6850 2100 6850
+Wire Wire Line
+	1900 6000 1900 6450
+Wire Wire Line
+	1900 6450 1900 6950
+Connection ~ 1900 6450
+Connection ~ 1900 6950
+Wire Wire Line
+	1900 6950 2100 6950
 $EndSCHEMATC

Commit message: Remove battery connector, charging circuit
Parts:
- removed C5: 47uF, Capacitor_SMD:C_0805_2012Metric, symbol device:C
- removed C7: 100nF, Capacitor_SMD:C_0805_2012Metric, symbol device:C
- removed CN2: TP4056, TP4056:TP4056, symbol tp4056:TP4056
- removed D1: SS36, Diode_SMD:D_SMA, symbol device:D_Schottky
- removed J3: Battery, Connector_Molex:Molex_PicoBlade_53048-0410_1x02_P1.25mm_Horizontal, symbol conn:Conn_01x02
- removed Q1: AO3401, Package_TO_SOT_SMD:SOT-23, symbol transistors:NTR2101P
- removed R2: 120k, Resistor_SMD:R_0805_2012Metric, symbol device:R
- removed R3: 390k, Resistor_SMD:R_0805_2012Metric, symbol device:R
- removed R8: 10k, Resistor_SMD:R_0805_2012Metric, symbol device:R
Connections:
- net labels added: FLASH, RST
- net labels removed: ADC, BAT+, BAT-, CHG+, HX+, VREG+
- wire segments 153 -> 113
- no-connect marks 9 -> 11
Other:
- note removed: "Battery Disconnector"
- note removed: "Battery Monitor"
- moved on the sheet: CN3, U2

Commit message: Better layout for load cell connectors, logo change
Changed lines of the file:
@@
 L conn:Conn_01x04 J12
 U 1 1 5B2A5EFA
-P 8900 5100
-F 0 "J12" H 8900 5300 50  0000 C CNN
-F 1 "Load Cell" H 8900 4800 50  0000 C CNN
-F 2 "Connector_Molex:Molex_PicoBlade_53048-0810_1x04_P1.25mm_Horizontal" H 8900 5100 50  0001 C CNN
-F 3 "" H 8900 5100 50  0001 C CNN
-	1    8900 5100
-	1    0    0    -1
+P 8900 5200
+F 0 "J12" H 8900 5400 50  0000 C CNN
+F 1 "Load Cell" H 8900 4900 50  0000 C CNN
+F 2 "Connector_Molex:Molex_PicoBlade_53048-0810_1x04_P1.25mm_Horizontal" H 8900 5200 50  0001 C CNN
+F 3 "" H 8900 5200 50  0001 C CNN
+	1    8900 5200
+	1    0    0    1
 $EndComp
 $Comp
@@
 L conn:Conn_01x04 J10
 U 1 1 5B504290
-P 8900 5700
-F 0 "J10" H 8900 5900 50  0000 C CNN
-F 1 "Load Cell" H 8900 5400 50  0000 C CNN
-F 2 "Connector_Molex:Molex_PicoBlade_53048-0810_1x04_P1.25mm_Horizontal" H 8900 5700 50  0001 C CNN
-F 3 "" H 8900 5700 50  0001 C CNN
-	1    8900 5700
-	1    0    0    -1
+P 8900 5800
+F 0 "J10" H 8900 6000 50  0000 C CNN
+F 1 "Load Cell" H 8900 5500 50  0000 C CNN
+F 2 "Connector_Molex:Molex_PicoBlade_53048-0810_1x04_P1.25mm_Horizontal" H 8900 5800 50  0001 C CNN
+F 3 "" H 8900 5800 50  0001 C CNN
+	1    8900 5800
+	1    0    0    1
 $EndComp
 $Comp
 L conn:Conn_01x04 J9
 U 1 1 5B5043D4
-P 8300 5700
-F 0 "J9" H 8300 5900 50  0000 C CNN
-F 1 "Load Cell" H 8300 5400 50  0000 C CNN
-F 2 "Connector_Molex:Molex_PicoBlade_53048-0810_1x04_P1.25mm_Horizontal" H 8300 5700 50  0001 C CNN
-F 3 "" H 8300 5700 50  0001 C CNN
-	1    8300 5700
-	1    0    0    -1
+P 8300 5800
+F 0 "J9" H 8300 6000 50  0000 C CNN
+F 1 "Load Cell" H 8300 5500 50  0000 C CNN
+F 2 "Connector_Molex:Molex_PicoBlade_53048-0810_1x04_P1.25mm_Horizontal" H 8300 5800 50  0001 C CNN
+F 3 "" H 8300 5800 50  0001 C CNN
+	1    8300 5800
+	1    0    0    1
 $EndComp
 $Comp
 L conn:Conn_01x04 J8
 U 1 1 5B504507
-P 8300 5100
-F 0 "J8" H 8300 5300 50  0000 C CNN
-F 1 "Load Cell" H 8300 4800 50  0000 C CNN
-F 2 "Connector_Molex:Molex_PicoBlade_53048-0810_1x04_P1.25mm_Horizontal" H 8300 5100 50  0001 C CNN
-F 3 "" H 8300 5100 50  0001 C CNN
-	1    8300 5100
-	1    0    0    -1
+P 8300 5200
+F 0 "J8" H 8300 5400 50  0000 C CNN
+F 1 "Load Cell" H 8300 4900 50  0000 C CNN
+F 2 "Connector_Molex:Molex_PicoBlade_53048-0810_1x04_P1.25mm_Horizontal" H 8300 5200 50  0001 C CNN
+F 3 "" H 8300 5200 50  0001 C CNN
+	1    8300 5200
+	1    0    0    1
 $EndComp
 Wire Wire Line

Commit message: Renumber parts to hit actual number of parts on board
Parts:
- renumbered C6 to C1, C4 to C2, C1 to C3, C8 to C4, C2 to C5, C3 to C6, CN3 to CN2, J4 to J1, J1 to J2, J8 to J3, J9 to J4, J12 to J5, J10 to J6, R9 to R2, R4 to R3, R5 to R4, R6 to R5, R7 to R6, U2 to U1, U1 to U2
Changed lines of the file:
@@
 Sheet 1 1
 Title "Libra Cervisiae PCB"
-Date "2018-07-23"
-Rev "0.1.0"
+Date "2018-08-09"
+Rev "0.1.2"
 Comp ""
 Comment1 ""
@@
 $EndDescr
 $Comp
-L regul:MCP1700-3302E_SOT23 U1
+L regul:MCP1700-3302E_SOT23 U2
 U 1 1 5B217881
 P 9050 2400
-F 0 "U1" H 8900 2525 50  0000 C CNN
+F 0 "U2" H 8900 2525 50  0000 C CNN
 F 1 "VREG" H 9050 2525 50  0000 L CNN
 F 2 "Package_TO_SOT_SMD:SOT-23" H 9050 2625 50  0001 C CNN
@@
 $EndComp
 $Comp
-L device:R R5
+L device:R R4
 U 1 1 5B21A80E
 P 6100 2750
-F 0 "R5" V 6180 2750 50  0000 C CNN
+F 0 "R4" V 6180 2750 50  0000 C CNN
 F 1 "10k" V 6100 2750 50  0000 C CNN
 F 2 "Resistor_SMD:R_0805_2012Metric" V 6030 2750 50  0001 C CNN
@@
 $EndComp
 $Comp
-L device:R R4
+L device:R R3
 U 1 1 5B21AA4B
 P 4000 2450
-F 0 "R4" V 4080 2450 50  0000 C CNN
+F 0 "R3" V 4080 2450 50  0000 C CNN
 F 1 "10k" V 4000 2450 50  0000 C CNN
 F 2 "Resistor_SMD:R_0805_2012Metric" V 3930 2450 50  0001 C CNN
@@
 $EndComp
 $Comp
-L device:R R7
+L device:R R6
 U 1 1 5B21AAD4
 P 6900 2650
-F 0 "R7" V 6980 2650 50  0000 C CNN
+F 0 "R6" V 6980 2650 50  0000 C CNN
 F 1 "10k" V 6900 2650 50  0000 C CNN
 F 2 "Resistor_SMD:R_0805_2012Metric" V 6830 2650 50  0001 C CNN
@@
 GND
 $Comp
-L device:R R6
+L device:R R5
 U 1 1 5B228DC8
 P 6350 2850
-F 0 "R6" V 6430 2850 50  0000 C CNN
+F 0 "R5" V 6430 2850 50  0000 C CNN
 F 1 "10k" V 6350 2850 50  0000 C CNN
 F 2 "Resistor_SMD:R_0805_2012Metric" V 6280 2850 50  0001 C CNN
@@
 $EndComp
 $Comp
-L device:C C3
+L device:C C6
 U 1 1 5B2296F3
 P 9750 2550
-F 0 "C3" H 9775 2650 50  0000 L CNN
+F 0 "C6" H 9775 2650 50  0000 L CNN
 F 1 "1uF" H 9775 2450 50  0000 L CNN
 F 2 "Capacitor_SMD:C_0805_2012Metric" H 9788 2400 50  0001 C CNN
@@
 $EndComp
 $Comp
-L ESP8266:ESP-12F U2
+L ESP8266:ESP-12F U1
 U 1 1 5B22CF91
 P 5050 2550
-F 0 "U2" H 5050 2450 50  0000 C CNN
+F 0 "U1" H 5050 2450 50  0000 C CNN
 F 1 "ESP-12F" H 5050 2650 50  0000 C CNN
 F 2 "ESP8266:ESP-12E" H 5050 2550 50  0001 C CNN
@@
 MCP1700
 $Comp
-L device:C C2
+L device:C C5
 U 1 1 5B241212
 P 8500 2550
-F 0 "C2" H 8525 2650 50  0000 L CNN
+F 0 "C5" H 8525 2650 50  0000 L CNN
 F 1 "1uF" H 8525 2450 50  0000 L CNN
 F 2 "Capacitor_SMD:C_0805_2012Metric" H 8538 2400 50  0001 C CNN
@@
 $EndComp
 $Comp
-L device:C C1
+L device:C C3
 U 1 1 5B2439F8
 P 5050 3750
-F 0 "C1" H 5075 3850 50  0000 L CNN
+F 0 "C3" H 5075 3850 50  0000 L CNN
 F 1 "47uF" H 5075 3650 50  0000 L CNN
 F 2 "Capacitor_SMD:C_0805_2012Metric" H 5088 3600 50  0001 C CNN
@@
 GND
 $Comp
-L power:PWR_FLAG #FLG02
+L power:PWR_FLAG #FLG01
 U 1 1 5B22D046
 P 3400 2650
-F 0 "#FLG02" H 3400 2725 50  0001 C CNN
+F 0 "#FLG01" H 3400 2725 50  0001 C CNN
 F 1 "PWR_FLAG" V 3450 2500 50  0000 C CNN
 F 2 "" H 3400 2650 50  0001 C CNN
@@
 $EndComp
 $Comp
-L conn:Conn_01x03 J4
+L conn:Conn_01x03 J1
 U 1 1 5B29B426
 P 2950 4900
-F 0 "J4" H 2950 5100 50  0000 C CNN
+F 0 "J1" H 2950 5100 50  0000 C CNN
 F 1 "Wort Temp" H 2950 4700 50  0000 C CNN
 F 2 "Connector_Molex:Molex_PicoBlade_53048-0610_1x03_P1.25mm_Horizontal" H 2950 4900 50  0001 C CNN
@@
 DS18B20s
 $Comp
-L hx711_breakout:HX711_BREAKOUT CN3
+L hx711_breakout:HX711_BREAKOUT CN2
 U 1 1 5B293345
 P 7550 5400
-F 0 "CN3" H 8050 4800 60  0000 C CNN
+F 0 "CN2" H 8050 4800 60  0000 C CNN
 F 1 "HX711_BREAKOUT" H 8050 5450 60  0000 C CNN
 F 2 "HX711:HX711-MINI" H 7550 5400 60  0001 C CNN
@@
 NoConn ~ 7550 4900
 $Comp
-L conn:Conn_01x04 J12
+L conn:Conn_01x04 J5
 U 1 1 5B2A5EFA
 P 8900 5200
-F 0 "J12" H 8900 5400 50  0000 C CNN
+F 0 "J5" H 8900 5400 50  0000 C CNN
 F 1 "Load Cell" H 8900 4900 50  0000 C CNN
 F 2 "Connector_Molex:Molex_PicoBlade_53048-0810_1x04_P1.25mm_Horizontal" H 8900 5200 50  0001 C CNN
@@
 $EndComp
 $Comp
-L device:C C4
+L device:C C2
 U 1 1 5B2A9325
 P 3350 5350
-F 0 "C4" V 3400 5200 50  0000 L CNN
+F 0 "C2" V 3400 5200 50  0000 L CNN
 F 1 "1uF" V 3500 5300 50  0000 L CNN
 F 2 "Capacitor_SMD:C_0805_2012Metric" H 3388 5200 50  0001 C CNN
@@
 USB+
 $Comp
-L device:C C6
+L device:C C1
 U 1 1 5B319707
 P 1700 2450
-F 0 "C6" H 1725 2550 50  0000 L CNN
+F 0 "C1" H 1725 2550 50  0000 L CNN
 F 1 "100nF" H 1800 2450 50  0000 L CNN
 F 2 "Capacitor_SMD:C_0805_2012Metric" H 1738 2300 50  0001 C CNN
@@
 	1700 2250 2050 2250
 $Comp
-L device:R R9
+L device:R R2
 U 1 1 5B4177F1
 P 3750 5350
-F 0 "R9" V 3830 5350 50  0000 C CNN
+F 0 "R2" V 3830 5350 50  0000 C CNN
 F 1 "10k" V 3750 5350 50  0000 C CNN
 F 2 "Resistor_SMD:R_0805_2012Metric" V 3680 5350 50  0001 C CNN
@@
 	6000 5250 6050 5250
 $Comp
-L device:C C8
+L device:C C4
 U 1 1 5B44D323
 P 6050 5050
-F 0 "C8" H 6050 4950 50  0000 L CNN
+F 0 "C4" H 6050 4950 50  0000 L CNN
 F 1 "1uF" H 5900 4950 50  0000 L CNN
 F 2 "Capacitor_SMD:C_0805_2012Metric" H 6088 4900 50  0001 C CNN
@@
 	6050 5250 6450 5250
 $Comp
-L conn:Conn_01x04 J10
+L conn:Conn_01x04 J6
 U 1 1 5B504290
 P 8900 5800
-F 0 "J10" H 8900 6000 50  0000 C CNN
+F 0 "J6" H 8900 6000 50  0000 C CNN
 F 1 "Load Cell" H 8900 5500 50  0000 C CNN
 F 2 "Connector_Molex:Molex_PicoBlade_53048-0810_1x04_P1.25mm_Horizontal" H 8900 5800 50  0001 C CNN
@@
 $EndComp
 $Comp
-L conn:Conn_01x04 J9
+L conn:Conn_01x04 J4
 U 1 1 5B5043D4
 P 8300 5800
-F 0 "J9" H 8300 6000 50  0000 C CNN
+F 0 "J4" H 8300 6000 50  0000 C CNN
 F 1 "Load Cell" H 8300 5500 50  0000 C CNN
 F 2 "Connector_Molex:Molex_PicoBlade_53048-0810_1x04_P1.25mm_Horizontal" H 8300 5800 50  0001 C CNN
@@
 $EndComp
 $Comp
-L conn:Conn_01x04 J8
+L conn:Conn_01x04 J3
 U 1 1 5B504507
 P 8300 5200
-F 0 "J8" H 8300 5400 50  0000 C CNN
+F 0 "J3" H 8300 5400 50  0000 C CNN
 F 1 "Load Cell" H 8300 4900 50  0000 C CNN
 F 2 "Connector_Molex:Molex_PicoBlade_53048-0810_1x04_P1.25mm_Horizontal" H 8300 5200 50  0001 C CNN
@@
 	3900 4900 4100 4900
 $Comp
-L conn:Conn_01x03 J1
+L conn:Conn_01x03 J2
 U 1 1 5B523E0B
 P 2950 5850
-F 0 "J1" H 2950 6050 50  0000 C CNN
+F 0 "J2" H 2950 6050 50  0000 C CNN
 F 1 "Board Temp" H 2950 5650 50  0000 C CNN
 F 2 "Package_TO_SOT_THT:TO-92" H 2950 5850 50  0001 C CNN

Commit message: Separate S- and E- planes for load cells, more bypass caps
Parts:
- added C4, C5: 100nF, Capacitor_SMD:C_0805_2012Metric, symbol device:C
- renumbered C4 to C6, C5 to C7, C6 to C8
Connections:
- wire segments 113 -> 122
Changed lines of the file:
@@
 $EndComp
 $Comp
-L device:C C6
+L device:C C8
 U 1 1 5B2296F3
 P 9750 2550
-F 0 "C6" H 9775 2650 50  0000 L CNN
+F 0 "C8" H 9775 2650 50  0000 L CNN
 F 1 "1uF" H 9775 2450 50  0000 L CNN
 F 2 "Capacitor_SMD:C_0805_2012Metric" H 9788 2400 50  0001 C CNN
@@
 MCP1700
 $Comp
-L device:C C5
+L device:C C7
 U 1 1 5B241212
 P 8500 2550
-F 0 "C5" H 8525 2650 50  0000 L CNN
+F 0 "C7" H 8525 2650 50  0000 L CNN
 F 1 "1uF" H 8525 2450 50  0000 L CNN
 F 2 "Capacitor_SMD:C_0805_2012Metric" H 8538 2400 50  0001 C CNN
@@
 Wire Wire Line
 	3850 2250 4100 2250
-Wire Wire Line
-	4050 2950 4050 3750
-Wire Wire Line
-	4050 3750 4900 3750
 Connection ~ 4050 2950
-Wire Wire Line
-	6200 3750 5200 3750
 Wire Wire Line
 	9750 2850 9750 2700
@@
 Wire Wire Line
 	8500 2700 8500 2850
-Wire Wire Line
-	6200 3750 6200 2950
 Connection ~ 6200 2950
 Wire Wire Line
@@
 	0    1    1    0
 $EndComp
-Wire Wire Line
-	6000 4900 6050 4900
-Wire Wire Line
-	6000 5250 6050 5250
-$Comp
-L device:C C4
+$Comp
+L device:C C6
 U 1 1 5B44D323
 P 6050 5050
-F 0 "C4" H 6050 4950 50  0000 L CNN
+F 0 "C6" H 6050 4950 50  0000 L CNN
 F 1 "1uF" H 5900 4950 50  0000 L CNN
 F 2 "Capacitor_SMD:C_0805_2012Metric" H 6088 4900 50  0001 C CNN
@@
 Text Label 6100 2650 0    60   ~ 0
 FLASH
+$Comp
+L device:C C4
+U 1 1 5B88593E
+P 5050 4050
+F 0 "C4" H 5075 4150 50  0000 L CNN
+F 1 "100nF" H 5075 3950 50  0000 L CNN
+F 2 "Capacitor_SMD:C_0805_2012Metric" H 5088 3900 50  0001 C CNN
+F 3 "" H 5050 4050 50  0001 C CNN
+	1    5050 4050
+	0    -1   -1   0
+$EndComp
+Wire Wire Line
+	4050 3900 4800 3900
+Wire Wire Line
+	4800 3900 4800 3750
+Wire Wire Line
+	4800 3750 4900 3750
+Wire Wire Line
+	4050 2950 4050 3900
+Wire Wire Line
+	4800 3900 4800 4050
+Wire Wire Line
+	4800 4050 4900 4050
+Connection ~ 4800 3900
+Wire Wire Line
+	5200 3750 5300 3750
+Wire Wire Line
+	5300 3750 5300 3900
+Wire Wire Line
+	5300 3900 6200 3900
+Wire Wire Line
+	6200 2950 6200 3900
+Wire Wire Line
+	5200 4050 5300 4050
+Wire Wire Line
+	5300 4050 5300 3900
+Connection ~ 5300 3900
+$Comp
+L device:C C5
+U 1 1 5B8B1FD8
+P 5650 5050
+F 0 "C5" H 5700 4950 50  0000 L CNN
+F 1 "100nF" H 5400 4950 50  0000 L CNN
+F 2 "Capacitor_SMD:C_0805_2012Metric" H 5688 4900 50  0001 C CNN
+F 3 "" H 5650 5050 50  0001 C CNN
+	1    5650 5050
+	1    0    0    -1
+$EndComp
+Wire Wire Line
+	5650 4900 6050 4900
+Wire Wire Line
+	5650 5250 5650 5200
+Wire Wire Line
+	5650 5250 6050 5250
 $EndSCHEMATC
